File: Eagle_files/NewWiring.brd (EAGLE design)
At the start: 103.8 x 85.1 mm, 60 parts, among them T1 PIN, T2 PIN

Commit message: Modified
Parts:
- added N1: CABLE, Kostas:CABLE
- added R12, R13, R14, R15, R16: RELAY, Kostas:RELAY
- moved H2 31.1 mm to (68.6, 6.35)
- moved T1 31.1 mm to (71.1, 6.35)
- moved B6 28.7 mm to (71.1, 12.7)
- moved B7 28.7 mm to (73.7, 12.7)
- moved CI2 28.7 mm to (63.5, 6.35)
- moved E11 28.7 mm to (63.5, 12.7)
- moved E12 28.7 mm to (66.0, 12.7)
- moved T2 28.7 mm to (66.0, 6.35)
- moved COLD_WATER_VALVE 28.1 mm to (43.2, 6.35)
- moved E9 26.2 mm to (61.0, 12.7)
- moved L3 26.2 mm to (61.0, 6.35)
- moved E4 23.7 mm to (50.8, 12.7)
- moved E5 23.7 mm to (53.3, 12.7)
- moved E7 23.7 mm to (58.4, 12.7)
- moved L1 23.7 mm to (53.3, 6.35)
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Connections:
- new net N$5: B6.P$1, B7.P$1, N1.P$1
- net D10: no longer HOT_WATER_VALVE.P$1
- net N$13: now also HOT_WATER_VALVE.P$1, N1.P$2; no longer B6.P$1, B7.P$1
Routing:
- net N$5: track 0.00 -> 30.5 mm
- net N$9: track 118.1 -> 147.3 mm
- net LIVE: track 106.7 -> 78.7 mm
- net N$16: track 105.4 -> 132.1 mm
- net N$11: track 125.7 -> 147.3 mm
- net N$13: track 17.8 -> 0.00 mm
- net N$6: track 95.2 -> 78.7 mm
- net N$47: track 69.1 -> 53.3 mm
- net N$25: track 29.2 -> 40.6 mm, vias 0 -> 2
- net N$15: track 129.5 -> 139.7 mm, vias 1 -> 2
- net NEUTRAL: track 120.7 -> 111.8 mm
- net N$42: track 29.2 -> 38.1 mm
- net N$23: track 47.0 -> 53.3 mm
- net N$24: track 57.1 -> 63.5 mm
- net N$43: track 39.4 -> 43.2 mm
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Other:
- board size 103.8 x 85.1 mm -> 102.5 x 77.5 mm

Commit message: Update
Parts:
- removed .S1, .S2, CA, CB, CI1, CI2, L1, L2, L3, MC1, MC2, MCC, MP1, MP2, MPC, S1, S2, T1, T2: PIN, Kostas:PIN
- removed H1, H2: PIN, Connectors:PIN
- added CAPACITOR: CAPACITOR, Kostas:CAPACITOR
- added HEATER: HEATER, Kostas:HEATER
- added MAIN_SWITCH: SWITCH, Kostas:SWITCH
- added PUMP: CI, Kostas:MOTOR-2
- added SPIN_MOTOR: MC, Kostas:MOTOR-3
- added THERMOSTAT: THERMOSTAT, Kostas:THERMOSTAT
- added U$1: LOCK, Kostas:LOCK
- added WASH_MOTOR: MP, Kostas:MOTOR-3
- moved COLD_WATER_VALVE 5.08 mm to (48.3, 6.35)
- moved HOT_WATER_VALVE 2.54 mm to (22.9, 6.35)
- moved PRESSURE-SWITCH_HA 2.54 mm to (88.9, 6.35)
Connections:
- removed net B7: B7.P$2, T1.P$1
- removed net C2: C2.P$2, MC2.P$1
- removed net C6: C6.P$2, MC1.P$1
- removed net N$27: B6.P$2, H2.P$1
- new net N$19: C6.P$2, SPIN_MOTOR.M1
- new net N$26: C2.P$2, SPIN_MOTOR.M3
- new net N$28: B7.P$2, THERMOSTAT.T1
- new net N$29: B6.P$2, HEATER.H1
- net C10: now also SPIN_MOTOR.MC, WASH_MOTOR.MC; no longer MCC.P$1, MPC.P$1
- net C11-OVERFLOW: now also PUMP.M1; no longer CI1.P$1
- net D2: now also WASH_MOTOR.M3; no longer MP2.P$1
- net D4: now also WASH_MOTOR.M1; no longer MP1.P$1
- net D6: now also CAPACITOR.C2; no longer CB.P$1
- net E11: now also PUMP.M3; no longer CI2.P$1
- net E5: now also U$1.N; no longer L1.P$1
- net N$1: now also MAIN_SWITCH.O1; no longer .S1.P$1
- net N$10: now also MAIN_SWITCH.I2; no longer S2.P$1
- net N$20: now also U$1.C; no longer L3.P$1
- net N$21: now also HEATER.H2; no longer H1.P$1
- net N$22: now also THERMOSTAT.T2; no longer T2.P$1
- net N$3: now also MAIN_SWITCH.O2, U$1.L; no longer .S2.P$1, L2.P$1
- net N$33: now also CAPACITOR.C1; no longer CA.P$1
- net N$8: now also MAIN_SWITCH.I1; no longer S1.P$1

Commit message: Added Cabling
Parts:
- added X1, X2, X3, X4, X5: DOMINO, Kostas:DOMINO
- moved R01 3.81 mm to (12.7, 43.2)
- moved R02 3.81 mm to (20.3, 43.2)
- moved R03 3.81 mm to (27.9, 43.2)
- moved R04 3.81 mm to (35.6, 43.2)
- moved R05 3.81 mm to (43.2, 43.2)
- moved R06 3.81 mm to (50.8, 43.2)
- moved R07 3.81 mm to (58.4, 43.2)
- moved R08 3.81 mm to (66.0, 43.2)
- moved R09 3.81 mm to (66.0, 68.6)
- moved R10 3.81 mm to (58.4, 68.6)
- moved R11 3.81 mm to (50.8, 68.6)
- moved R12 3.81 mm to (43.2, 68.6)
- moved R13 3.81 mm to (35.6, 68.6)
- moved R14 3.81 mm to (27.9, 68.6)
- moved R15 3.81 mm to (20.3, 68.6)
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Connections:
- new net N$27: E2.P$1, R09.R, X1.P$2
- new net N$30: D6.P$1, R09.T, X2.P$2
- new net N$31: R11.C, X2.P$1
- new net N$32: R07.C, R08.C, X3.P$2
- new net N$35: R04.C, R05.C, X5.P$2
- net N$15: now also R10.C, X1.P$1; no longer D6.P$1, R09.T, R11.C
- net N$16: now also R02.T, R03.T, X4.P$2; no longer E2.P$1, R09.R, R10.C
- net NEUTRAL: now also X3.P$1; no longer R07.C, R08.C
- net PHASE3: now also X4.P$1, X5.P$1; no longer R02.T, R03.T, R04.C, R05.C
Routing:
- net N$15: track 139.7 -> 10.2 mm, vias 2 -> 0
- net N$30: track 0.00 -> 124.8 mm, vias 0 -> 3
- net N$27: track 0.00 -> 117.1 mm, vias 0 -> 3
- net N$16: track 132.1 -> 26.9 mm, vias 3 -> 1
- net N$14: track 0.00 -> 90.2 mm, vias 0 -> 4
- net N$7: track 0.00 -> 87.6 mm, vias 0 -> 4
- net PHASE3: track 81.3 -> 49.8 mm, vias 1 -> 2
- net N$32: track 0.00 -> 26.9 mm, vias 0 -> 1
- net N$35: track 0.00 -> 26.9 mm, vias 0 -> 1
- net N$31: track 0.00 -> 26.7 mm, vias 0 -> 1
- net N$9: track 147.3 -> 128.3 mm, vias 1 -> 4
- net N$11: track 147.3 -> 133.4 mm, vias 1 -> 4
- net NEUTRAL: track 111.8 -> 98.1 mm
- net N$12: track 68.6 -> 58.4 mm, vias 2 -> 4
- net N$5: track 30.5 -> 21.8 mm
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Other:
- board size 102.5 x 77.5 mm -> 102.5 x 76.2 mm

Commit message: Update
Routing:
- net N$7: track 87.6 -> 153.7 mm
- net N$14: track 90.2 -> 151.1 mm
- net N$9: track 128.3 -> 133.4 mm
Changed lines of the file:
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@@
 <contactref element="D2" pad="P$1"/>
 <wire x1="48.26" y1="67.31" x2="48.26" y2="76.2" width="0.4064" layer="1"/>
-<wire x1="48.26" y1="76.2" x2="31.75" y2="76.2" width="0.4064" layer="16"/>
-<via x="31.75" y="76.2" extent="1-16" drill="0.0254" diameter="0.127"/>
-<wire x1="31.75" y1="76.2" x2="31.75" y2="19.05" width="0.4064" layer="1"/>
-<wire x1="31.75" y1="19.05" x2="33.02" y2="19.05" width="0.4064" layer="16"/>
+<wire x1="48.26" y1="76.2" x2="1.27" y2="76.2" width="0.4064" layer="16"/>
+<via x="1.27" y="76.2" extent="1-16" drill="0.0254" diameter="0.127"/>
+<wire x1="1.27" y1="76.2" x2="1.27" y2="19.05" width="0.4064" layer="1"/>
+<wire x1="1.27" y1="19.05" x2="33.02" y2="19.05" width="0.4064" layer="16"/>
 <wire x1="33.02" y1="19.05" x2="33.02" y2="12.7" width="0.4064" layer="1"/>
-<via x="31.75" y="19.05" extent="1-16" drill="0.0254" diameter="0.127"/>
+<via x="1.27" y="19.05" extent="1-16" drill="0.0254" diameter="0.127"/>
 <via x="33.02" y="19.05" extent="1-16" drill="0.0254" diameter="0.127"/>
 <via x="48.26" y="76.2" extent="1-16" drill="0.0254" diameter="0.127"/>
@@
 <contactref element="R10" pad="R"/>
 <contactref element="D4" pad="P$1"/>
-<wire x1="55.88" y1="67.31" x2="55.88" y2="74.93" width="0.4064" layer="1"/>
-<via x="55.88" y="74.93" extent="1-16" drill="0.0254" diameter="0.127"/>
-<wire x1="55.88" y1="74.93" x2="39.37" y2="74.93" width="0.4064" layer="16"/>
-<via x="39.37" y="74.93" extent="1-16" drill="0.0254" diameter="0.127"/>
-<wire x1="39.37" y1="74.93" x2="39.37" y2="21.59" width="0.4064" layer="1"/>
-<wire x1="39.37" y1="21.59" x2="38.1" y2="21.59" width="0.4064" layer="16"/>
+<wire x1="55.88" y1="67.31" x2="55.88" y2="73.66" width="0.4064" layer="1"/>
+<via x="55.88" y="73.66" extent="1-16" drill="0.0254" diameter="0.127"/>
+<wire x1="55.88" y1="73.66" x2="3.81" y2="73.66" width="0.4064" layer="16"/>
+<via x="3.81" y="73.66" extent="1-16" drill="0.0254" diameter="0.127"/>
+<wire x1="3.81" y1="73.66" x2="3.81" y2="21.59" width="0.4064" layer="1"/>
+<wire x1="3.81" y1="21.59" x2="38.1" y2="21.59" width="0.4064" layer="16"/>
 <wire x1="38.1" y1="21.59" x2="38.1" y2="12.7" width="0.4064" layer="1"/>
-<via x="39.37" y="21.59" extent="1-16" drill="0.0254" diameter="0.127"/>
+<via x="3.81" y="21.59" extent="1-16" drill="0.0254" diameter="0.127"/>
 <via x="38.1" y="21.59" extent="1-16" drill="0.0254" diameter="0.127"/>
 </signal>
@@
 <contactref element="R11" pad="T"/>
 <contactref element="C2" pad="P$1"/>
-<wire x1="3.81" y1="73.66" x2="53.34" y2="73.66" width="0.4064" layer="16"/>
-<via x="53.34" y="73.66" extent="1-16" drill="0.0254" diameter="0.254"/>
-<wire x1="53.34" y1="73.66" x2="53.34" y2="67.31" width="0.4064" layer="1"/>
+<wire x1="2.54" y1="74.93" x2="53.34" y2="74.93" width="0.4064" layer="16"/>
+<via x="53.34" y="74.93" extent="1-16" drill="0.0254" diameter="0.254"/>
+<wire x1="53.34" y1="74.93" x2="53.34" y2="67.31" width="0.4064" layer="1"/>
 <wire x1="15.24" y1="12.7" x2="15.24" y2="20.32" width="0.4064" layer="1"/>
-<wire x1="15.24" y1="20.32" x2="3.81" y2="20.32" width="0.4064" layer="16"/>
-<wire x1="3.81" y1="20.32" x2="3.81" y2="73.66" width="0.4064" layer="1"/>
-<via x="3.81" y="20.32" extent="1-16" drill="0.0254" diameter="0.127"/>
-<via x="3.81" y="73.66" extent="1-16" drill="0.0254" diameter="0.127"/>
+<wire x1="15.24" y1="20.32" x2="2.54" y2="20.32" width="0.4064" layer="16"/>
+<wire x1="2.54" y1="20.32" x2="2.54" y2="74.93" width="0.4064" layer="1"/>
+<via x="2.54" y="20.32" extent="1-16" drill="0.0254" diameter="0.127"/>
+<via x="2.54" y="74.93" extent="1-16" drill="0.0254" diameter="0.127"/>
 <via x="15.24" y="20.32" extent="1-16" drill="0.0254" diameter="0.127"/>
 </signal>

Commit message: Improved
Parts:
- moved X1 14.0 mm to (72.4, 77.5)
- moved X2 8.98 mm to (72.4, 80.0)
- moved E11 2.54 mm to (66.0, 12.7)
- moved E9 2.54 mm to (63.5, 12.7)
- moved E12 2.54 mm to (68.6, 12.7)
- moved N1 2.54 mm to (76.2, 12.7)
Routing:
- net N$15: track 10.2 -> 24.1 mm, vias 0 -> 1
- net N$31: track 26.7 -> 34.3 mm
- net N$12: track 58.4 -> 66.0 mm
- net N$27: track 117.1 -> 119.7 mm, vias 3 -> 4
- net N$5: track 21.8 -> 19.3 mm
- net LIVE: track 73.0 -> 75.5 mm
- net N$30: vias 3 -> 4
